Commit message: done

File: ros_gz_example_description/models/manipulator/model.urdf (robot description, URDF)
Before this commit: robot manipulator, 5 links, 4 joints
Joints:
- joint joint_2: axis 0 -1 0 -> 0 0 1; origin xyz=0.0 0 0.05 rpy=0 1.5708 0 -> xyz=0.0 0 0.05 rpy=1.57 0 0
- joint joint_3: axis 0 -1 0 -> 0 0 1; origin xyz=0 0 0.2 rpy=0 0 0 -> xyz=0.2 0 0.0 rpy=0 0 0

Commit message: done. dynamics, jacobian

File: ros_gz_example_description/models/manipulator/model.urdf (robot description, URDF)
Before this commit: robot manipulator, 5 links, 4 joints
Links:
- added link link_EE; visual sphere radius=0.03
Joints:
- added joint joint_EE: type fixed, parent link_3, child link_EE, origin xyz=0.2 0.0 0.0 rpy=0 0 0

Commit message: Let's align force sensor frame

File: ros_gz_example_description/models/manipulator/model.urdf (robot description, URDF)
Before this commit: robot manipulator, 6 links, 5 joints
Joints:
- joint joint_EE: axis (none) -> 0 0 1; limit (none) -> lower=-1.57 upper=1.57 effort=100 velocity=10.0

Commit message: sdf urdf visual

File: ros_gz_example_description/models/manipulator/model.urdf (robot description, URDF)
Before this commit: robot manipulator, 6 links, 5 joints
Links:
- link link_drone: geometry visual mesh filename=package://ros_gz_example_description/models/manipulator/mes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 scale=0.001 0.001 0.001

Commit message: state_dot is body. EE_vel is right. wall defined

File: ros_gz_example_description/models/manipulator/model.urdf (robot description, URDF)
Before this commit: robot manipulator, 6 links, 5 joints
Links:
- link link_drone: geometry visual mesh filename=package://ros_gz_example_description/models/manipulator/mes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 scale=0.00085 0.00085 0.00085

Commit message: 민재는 받아라.

File: ros_gz_example_description/models/manipulator/model.urdf (robot description, URDF)
Before this commit: robot manipulator, 6 links, 5 joints
Links:
- removed link link_1
- removed link link_2
- removed link link_3
- removed link link_EE
- added link curvature_link; visual mesh filename=package://ros_gz_example_description/models/manipulator/mes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 scale=0.004 0.004 0.004
- added link link_ee, mass 0.1; visual mesh filename=package://ros_gz_example_description/models/manipulator/mes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 scale=0.001 0.001 0.001
- added link sphere_link; visual mesh filename=package://ros_gz_example_description/models/manipulator/mes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 scale=0.006 0.006 0.006
- link link_drone: geometry visual mesh filename=package://ros_gz_example_description/models/manipulator/mes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 scale=0.001 0.001 0.001
Joints:
- removed joint joint_1
- removed joint joint_2
- removed joint joint_3
- removed joint joint_EE
- added joint drone_to_ee: type fixed, parent link_drone, child link_ee, origin xyz=0 0 0 rpy=0 0 0
- added joint world_to_curvature: type fixed, parent world, child curvature_link, origin xyz=1.5 0.8 0 rpy=0 0 0
- added joint world_to_sphere: type fixed, parent world, child sphere_link, origin xyz=1.5 -1.2 0 rpy=0 0 0
